File: Battery/Battery.sch (KiCad schematic (older format))
At the start: 1 part

Commit message: Pabeigts
Parts:
- BT1: footprint (none) -> Battery_Holder:SMTU2032
Changed lines of the file:
@@
 F 0 "BT1" H 1068 1246 50  0000 L CNN
 F 1 "Battery_Cell" H 1068 1155 50  0000 L CNN
-F 2 "" V 950 1210 50  0001 C CNN
+F 2 "Battery_Holder:SMTU2032" V 950 1210 50  0001 C CNN
 F 3 "~" V 950 1210 50  0001 C CNN
 	1    950  1150

Commit message: Md
Parts:
- BT1: footprint Battery_Holder:SMTU2032 -> Battery_Holder:4u-2101G4D405-H
Changed lines of the file:
@@
 F 0 "BT1" H 1068 1246 50  0000 L CNN
 F 1 "Battery_Cell" H 1068 1155 50  0000 L CNN
-F 2 "Battery_Holder:SMTU2032" V 950 1210 50  0001 C CNN
+F 2 "Battery_Holder:4u-2101G4D405-H" V 950 1210 50  0001 C CNN
 F 3 "~" V 950 1210 50  0001 C CNN
 	1    950  1150
