File: Matricas_dala/Led_matrica.kicad_pcb (KiCad board)
At the start: 2 copper layers, 260 x 75 mm, 314 parts, among them J1 Screw_Terminal_01x08, U1 74HC595, U10 BC807RA, U11 BC807RA, U12 BC807RA, U13 BC807RA, U14 BC807RA, U15 BC807RA, U16 BC807RA, U17 BC807RA, U18 BC807RA, U19 BC807RA, U2 74HC595, U20 BC807RA, U3 74HC595, U4 74HC595, U6 74HC595, U7 74HC595, U8 74HC595, U9 BC807RA

Commit message: Kursa darbs
Parts:
- added REF**: MountingHole_2.5mm_Pad, MountingHole:MountingHole_2.5mm_Pad, F.Cu at (260.5, 19.5)
- added REF**: MountingHole_2.5mm_Pad, MountingHole:MountingHole_2.5mm_Pad, F.Cu at (260.3, 85.9)
- added REF**: MountingHole_2.5mm_Pad, MountingHole:MountingHole_2.5mm_Pad, F.Cu at (9.30, 19.9)
- R17: value 1k -> 150
- R18, R19: value 1k -> 100
- R20, R23: value R_Small -> 150
- R21, R22, R24: value R_Small -> 100
Connections:
- U10 pad 3: R4 -> R2
- U10 pad 6: R3 -> B1
- U11 pad 3: R6 -> B2
- U11 pad 6: R5 -> G2
- U12 pad 3: R8 -> G3
- U12 pad 6: R7 -> R3
- U13 pad 3: G2 -> R4
- U13 pad 6: G1 -> B3
- U14 pad 3: G4 -> B4
- U14 pad 6: G3 -> G4
- U15 pad 3: G6 -> G5
- U15 pad 6: G5 -> R5
- U16 pad 3: G8 -> R6
- U16 pad 6: G7 -> B5
- U17 pad 3: B2 -> B6
- U17 pad 6: B1 -> G6
- U18 pad 3: B4 -> G7
- U18 pad 6: B3 -> R7
- U19 pad 3: B6 -> R8
- U19 pad 6: B5 -> B7
- U20 pad 6: B7 -> G8
- U9 pad 3: R2 -> G1
Routing:
- net Vcc: track 127.6 -> 133.9 mm, vias 26 -> 27
- net Output_Enable: track 254.0 -> 252.1 mm
- net Net-(R32-Pad2): track 9.30 -> 7.57 mm
- net Net-(R30-Pad2): track 5.26 -> 6.91 mm
- net Net-(R29-Pad2): track 4.03 -> 4.93 mm
- net Net-(R24-Pad1): track 5.33 -> 6.19 mm, vias 0 -> 1
- net Net-(R37-Pad1): track 9.59 -> 10.2 mm, vias 0 -> 1
- net Net-(R35-Pad1): track 8.76 -> 9.33 mm, vias 0 -> 1
- net Net-(R28-Pad1): track 4.57 -> 5.03 mm, vias 0 -> 1
- net Net-(R38-Pad1): track 3.75 -> 4.19 mm, vias 0 -> 1
- net Net-(R19-Pad1): track 9.83 -> 10.3 mm, vias 0 -> 1
- net Net-(R20-Pad1): track 5.74 -> 5.33 mm, vias 0 -> 1
- net Net-(R29-Pad1): track 9.33 -> 9.73 mm, vias 0 -> 1
- net Net-(R31-Pad1): track 9.19 -> 9.56 mm, vias 0 -> 1
- net Net-(R27-Pad1): track 8.92 -> 9.24 mm, vias 0 -> 1
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