File: Matricas_dala/Vadiba.sch (KiCad schematic (older format))
At the start: 58 parts, among them J1 Screw_Terminal_01x08, U1 74HC595, U10 BC807RA, U11 BC807RA, U12 BC807RA, U13 BC807RA, U14 BC807RA, U15 BC807RA, U16 BC807RA, U17 BC807RA, U18 BC807RA, U19 BC807RA, U2 74HC595, U20 BC807RA, U3 74HC595, U4 74HC595, U6 74HC595, U7 74HC595, U8 74HC595, U9 BC807RA

Commit message: Kursa darbs
Parts:
- removed R32, R33, R34, R35, R36, R37, R38, R39, R40: R_Small, Resistor_SMD:R_0805_2012Metric, symbol Device:R_Small
- added R10, R12, R13, R15, R9: 100, Resistor_SMD:R_0805_2012Metric, symbol Device:R_Small
- added R11, R14, R16, R8: 150, Resistor_SMD:R_0805_2012Metric, symbol Device:R_Small
- R25, R26, R28, R29, R31: value R_Small -> 100
- R27, R30: value R_Small -> 150
Connections:
- net B1: now also U10.6 (C); no longer U17.6 (C)
- net B2: now also U11.3 (C); no longer U17.3 (C)
- net B3: now also U13.6 (C); no longer U18.6 (C)
- net B4: now also U14.3 (C); no longer U18.3 (C)
- net B5: now also U16.6 (C); no longer U19.6 (C)
- net B6: now also U17.3 (C); no longer U19.3 (C)
- net B7: now also U19.6 (C); no longer U20.6 (C)
- net G1: now also U9.3 (C); no longer U13.6 (C)
- net G2: now also U11.6 (C); no longer U13.3 (C)
- net G3: now also U12.3 (C); no longer U14.6 (C)
- net G4: now also U14.6 (C); no longer U14.3 (C)
- net G5: now also U15.3 (C); no longer U15.6 (C)
- net G6: now also U17.6 (C); no longer U15.3 (C)
- net G7: now also U18.3 (C); no longer U16.6 (C)
- net G8: now also U20.6 (C); no longer U16.3 (C)
- net R2: now also U10.3 (C); no longer U9.3 (C)
- net R3: now also U12.6 (C); no longer U10.6 (C)
- net R4: now also U13.3 (C); no longer U10.3 (C)
- net R5: now also U15.6 (C); no longer U11.6 (C)
- net R6: now also U16.3 (C); no longer U11.3 (C)
- net R7: now also U18.6 (C); no longer U12.6 (C)
- net R8: now also U19.3 (C); no longer U12.3 (C)
- net at U7.1 (QB): now also R9.2; no longer R26.2
- net at U7.15 (QA): now also R8.2; no longer R25.2
- net at U7.2 (QC): now also R10.2; no longer R27.2
- net at U7.3 (QD): now also R11.2; no longer R28.2
- net at U7.4 (QE): now also R12.2; no longer R29.2
- net at U7.5 (QF): now also R13.2; no longer R30.2
- net at U7.6 (QG): now also R14.2; no longer R31.2
- net at U7.7 (QH): now also R15.2
- net at U8.1 (QB): now also R25.2
- net at U8.15 (QA): now also R16.2
- net at U8.2 (QC): now also R26.2
- net at U8.3 (QD): now also R27.2
- net at U8.4 (QE): now also R28.2
- net at U8.5 (QF): now also R29.2
- net at U8.6 (QG): now also R30.2
- net at U8.7 (QH): now also R31.2
- net at U13.2 (B): now also R8.1; no longer R25.1
- net at U13.5 (B): now also R9.1; no longer R26.1
- net at U14.2 (B): now also R10.1; no longer R27.1
- net at U14.5 (B): now also R11.1; no longer R28.1
- net at U15.2 (B): now also R12.1; no longer R29.1
- net at U15.5 (B): now also R13.1; no longer R30.1
- net at U16.2 (B): now also R14.1; no longer R31.1
- net at U16.5 (B): now also R15.1
- net at U17.2 (B): now also R16.1
- net at U17.5 (B): now also R25.1
- net at U18.2 (B): now also R26.1
- net at U18.5 (B): now also R27.1
- net at U19.2 (B): now also R28.1
- net at U19.5 (B): now also R29.1
- net at U20.2 (B): now also R30.1
- net at U20.5 (B): now also R31.1
